File: hardware/piTrex.sch (KiCad schematic (older format))
At the start: 14 parts, among them CON1 vectrex-edge-connector, J1 Raspberry_Pi_2_3, J2 Test, J3 SPI Sel, Q1 DMG2305UX, U1 DMMT5401, U2 XC9572XL-VQFP44

Commit message: Initial gateware
Parts:
- C1, C2, C3: LCSC (none) -> C106243
- J1: LCSC (none) -> C132132
- Q1: LCSC (none) -> C150470
- R1, R2: LCSC (none) -> C84376
- RN1: LCSC (none) -> C102673
- U1: LCSC (none) -> C154733
Connections:
- net labels added: CLOCK, IP_BUSY, IP_COMMAND, IP_RESET
- net labels removed: PI_PB6, ~PI_IRQ
- wire segments 102 -> 107
- no-connect marks 22 -> 20
Changed lines of the file:
@@
 F 2 "piTrex:PiZeroHat" H 2950 6600 50  0001 C CNN
 F 3 "" H 2000 5200 50  0001 C CNN
+F 4 "C132132" H 1950 5350 50  0001 C CNN "LCSC"
 	1    1950 5350
 	1    0    0    -1
@@
 Text Label 9150 2500 2    50   ~ 0
 ~E
-Text Label 9150 2400 2    50   ~ 0
-~HALT
 $Comp
 L Device:C C3
@@
 F 2 "Capacitor_SMD:C_0805_2012Metric_Pad1.15x1.40mm_HandSolder" H 5238 5200 50  0001 C CNN
 F 3 "" H 5200 5350 50  0001 C CNN
+F 4 "C106243" H 5200 5350 50  0001 C CNN "LCSC"
 	1    5200 5350
 	1    0    0    -1
@@
 F 2 "Capacitor_SMD:C_0805_2012Metric_Pad1.15x1.40mm_HandSolder" H 5038 5200 50  0001 C CNN
 F 3 "" H 5000 5350 50  0001 C CNN
+F 4 "C106243" H 5000 5350 50  0001 C CNN "LCSC"
 	1    5000 5350
 	1    0    0    -1
@@
 F 2 "Capacitor_SMD:C_0805_2012Metric_Pad1.15x1.40mm_HandSolder" H 4838 5200 50  0001 C CNN
 F 3 "" H 4800 5350 50  0001 C CNN
+F 4 "C106243" H 4800 5350 50  0001 C CNN "LCSC"
 	1    4800 5350
 	1    0    0    -1
@@
 F 2 "Resistor_SMD:R_Array_Concave_4x0603" V 8475 4800 50  0001 C CNN
 F 3 "" H 8200 4800 50  0001 C CNN
+F 4 "C102673" V 8200 4800 50  0001 C CNN "LCSC"
 	1    8200 4800
 	1    0    0    1
@@
 F 2 "Package_TO_SOT_SMD:SOT-23_Handsoldering" H 1550 1500 50  0001 C CNN
 F 3 "" H 1350 1400 50  0001 C CNN
+F 4 "C150470" V 1350 1400 50  0001 C CNN "LCSC"
 	1    1350 1400
 	0    -1   -1   0
@@
 F 2 "Package_TO_SOT_SMD:SOT-23-6_Handsoldering" H 1300 1850 60  0001 C CNN
 F 3 "" H 1300 1850 60  0000 C CNN
+F 4 "C154733" V 1300 1850 50  0001 C CNN "LCSC"
 	1    1300 1850
 	1    0    0    -1
@@
 F 2 "Resistor_SMD:R_0805_2012Metric_Pad1.15x1.40mm_HandSolder" V 1030 2700 50  0001 C CNN
 F 3 "" H 1100 2700 50  0001 C CNN
+F 4 "C84376" V 1100 2700 50  0001 C CNN "LCSC"
 	1    1100 2700
 	1    0    0    -1
@@
 F 2 "Resistor_SMD:R_0805_2012Metric_Pad1.15x1.40mm_HandSolder" V 1530 2700 50  0001 C CNN
 F 3 "" H 1600 2700 50  0001 C CNN
+F 4 "C84376" V 1600 2700 50  0001 C CNN "LCSC"
 	1    1600 2700
 	1    0    0    -1
@@
 Wire Wire Line
 	1600 2500 1600 2550
-Text Label 2850 4550 0    50   ~ 0
-~PI_IRQ
-Text Label 2850 4450 0    50   ~ 0
-PI_PB6
 Connection ~ 2250 6800
 $Comp
@@
 Wire Wire Line
 	4050 2800 4400 2800
-Text Label 5500 2700 2    50   ~ 0
-~HALT
 Text Label 5500 2550 2    50   ~ 0
 A7
@@
 NoConn ~ 1050 5550
 NoConn ~ 1050 5650
-NoConn ~ 1050 5750
 NoConn ~ 1050 6050
 NoConn ~ 1050 6150
@@
 NoConn ~ 2850 4950
 NoConn ~ 2850 4850
-NoConn ~ 2850 4650
 NoConn ~ 2850 4550
 NoConn ~ 2850 4450
 NoConn ~ 2150 4050
 NoConn ~ 1850 4050
+$Comp
+L power:GND #PWR?
+U 1 1 5B8558EE
+P 8650 2450
+F 0 "#PWR?" H 8650 2200 50  0001 C CNN
+F 1 "GND" H 8655 2277 50  0000 C CNN
+F 2 "" H 8650 2450 50  0001 C CNN
+F 3 "" H 8650 2450 50  0001 C CNN
+	1    8650 2450
+	1    0    0    -1
+$EndComp
+Wire Wire Line
+	9150 2400 8650 2400
+Wire Wire Line
+	8650 2400 8650 2450
+Text Label 5500 2700 2    50   ~ 0
+CLOCK
+Text Label 2850 4650 0    50   ~ 0
+CLOCK
+Text Label 150  4750 2    50   ~ 0
+IP_BUSY
+Text Label 150  5750 2    50   ~ 0
+IP_RESET
+Text Label 150  5250 2    50   ~ 0
+IP_COMMAND
+Wire Wire Line
+	1050 4750 150  4750
+Wire Wire Line
+	1050 5250 150  5250
+Wire Wire Line
+	1050 5750 150  5750
 $EndSCHEMATC
